File: hardware/motor-driver/motor-driver.kicad_sch (KiCad schematic)
At the start: 18 parts, among them J1 48V_BUS_IN (XT60), J2 MOTOR_PHASES, J3 SPI_CTRL (MCU), Q1H IRF2907, Q1L IRF2907, Q2H IRF2907, Q2L IRF2907, Q3H IRF2907, Q3L IRF2907, U1 DRV8353RS

Commit message: hardware: regenerate KiCad schematics with correct KiCad 7 syntax
Previous schematics had multiple parser errors:
- (label (text "X") ...) should be (label "X" ...)
- pin instances used names not numbers
- UTF-8 BOM byte from PowerShell Set-Content

Added gen_schematics.py Python generator as source-of-truth.
All three .kicad_sch files now pass: no BOM, starts with '(',
balanced parentheses, correct KiCad 7 S-expression format.

Co-Authored-By: Claude Opus 4.7 (1M context) <noreply@anthropic.com>
Parts:
- removed C_BOOT_A, C_BOOT_B, C_BOOT_C: 100n, symbol C_Generic
- removed C_VM1: 10u/63V, symbol C_Generic
- removed C_VM2: 100n/63V, symbol C_Generic
- removed RSH_A, RSH_B, RSH_C: 5m / 2W, symbol R_Shunt
- J1: value 48V_BUS_IN (XT60) -> 48V_IN; footprint (none) -> Connector_PinHeader_2.54mm:PinHeader_1x02_P2.54mm_Vertical
- J2: footprint (none) -> Connector_PinHeader_2.54mm:PinHeader_1x03_P2.54mm_Vertical
- J3: value SPI_CTRL (MCU) -> SPI_CTRL; footprint (none) -> Connector_PinHeader_2.54mm:PinHeader_1x06_P2.54mm_Vertical
- Q1H, Q1L, Q2H, Q2L, Q3H, Q3L: footprint (none) -> Package_TO_SOT_THT:TO-247-3_Vertical
Connections:
- net ['text', 'DRV_ENABLE']: no longer names the net of U1.3 (DVDD)
- net ['text', 'GH_A']: no longer names the net of U1.17 (SH_A)
- net ['text', 'GH_B']: no longer names the net of U1.14 (GL_B)
- net ['text', 'GH_C']: no longer names the net of U1.11 (GH_A)
- net ['text', 'GL_A']: no longer names the net of U1.16 (GL_C)
- net ['text', 'GL_B']: no longer names the net of U1.13 (GH_B)
- net ['text', 'SPI_SCLK']: no longer names the net of U1.1 (VM)
- net ['text', 'SPI_SCS']: no longer names the net of U1.2 (VCP)
Other:
- note added: "NOTE: One board per joint (x7 total). U2..U7 = identical DRV8353RS."
- title: Motor Driver — 7-DoF Arm Joint -> Motor Driver - 7-DoF Arm Joint
