File: hardware/power-distribution/power-distribution.kicad_sch (KiCad schematic)
At the start: 15 parts, among them J1 48V_BATT_IN (XT60), J2 VM_OUT (to motor drivers, x7), J3 +5V_OUT, J4 +3V3_OUT, Q1 IRF2907 (E-stop), U1 LMR36520 (48V→5V/3A), U2 TLV1117-33 (5V→3.3V/800mA)

Commit message: hardware: regenerate KiCad schematics with correct KiCad 7 syntax
Previous schematics had multiple parser errors:
- (label (text "X") ...) should be (label "X" ...)
- pin instances used names not numbers
- UTF-8 BOM byte from PowerShell Set-Content

Added gen_schematics.py Python generator as source-of-truth.
All three .kicad_sch files now pass: no BOM, starts with '(',
balanced parentheses, correct KiCad 7 S-expression format.

Co-Authored-By: Claude Opus 4.7 (1M context) <noreply@anthropic.com>
Parts:
- removed C_IN1: 100u/63V, symbol Cap
- removed C_IN2: 100n/63V, symbol Cap
- removed C_OUT1: 220u/10V, symbol Cap
- removed C_OUT2: 100n/10V, symbol Cap
- removed D1: P6KE58A (58V clamp), symbol D_TVS
- removed J1: 48V_BATT_IN (XT60), symbol Conn2
- removed J2: VM_OUT (to motor drivers, x7), symbol Conn2
- removed J3: +5V_OUT, symbol Conn2
- removed J4: +3V3_OUT, symbol Conn2
- removed L1: 22u / 3A, symbol Inductor
- removed Q1: IRF2907 (E-stop), symbol IRF2907_estop
- removed R_GATE: 10k, symbol Cap
- removed U2: TLV1117-33 (5V→3.3V/800mA), symbol TLV1117
- added D1: P6KE58A, Diode_THT:D_DO-15_P12.70mm_Horizontal, symbol D_TVS_P6KE58A
- added J1: 48V_BATT_IN (XT60), Connector_PinHeader_2.54mm:PinHeader_1x02_P2.54mm_Vertical, symbol Conn_2pin
- added J2: VM_OUT (48V to drivers), Connector_PinHeader_2.54mm:PinHeader_1x02_P2.54mm_Vertical, symbol Conn_2pin
- added J3: +5V_OUT, Connector_PinHeader_2.54mm:PinHeader_1x02_P2.54mm_Vertical, symbol Conn_2pin
- added J4: +3V3_OUT, Connector_PinHeader_2.54mm:PinHeader_1x02_P2.54mm_Vertical, symbol Conn_2pin
- added Q1: IRF2907, Package_TO_SOT_THT:TO-247-3_Vertical, symbol IRF2907_ESTOP
- added U2: TLV1117-33, Package_TO_SOT_THT:TO-252-2, symbol TLV1117-33
- F1: value 32A / Littelfuse 0218032 -> 32A/250V; footprint (none) -> Fuse:Fuse_Littelfuse_NANO2_154Series_L6.1mm_W2.6mm_P10.9mm
- U1: value LMR36520 (48V→5V/3A) -> LMR36520; footprint (none) -> Package_TO_SOT_SMD:SOT-23-8
Connections:
- net ['text', '48V_FUSED']: no longer names the net of F1.2 (K)
- net ['text', '48V_RAW']: no longer names the net of F1.1 (A)
- net ['text', 'SW_NODE']: no longer names the net of U1.5 (SW)
Other:
- note added: "LMR36520: 48V->5V/3A buck | TLV1117-33: 5V->3.3V/800mA LDO"
- note added: "Power tree: 48V battery -> 32A fuse -> TVS clamp -> E-stop FET -> motor drivers"
- title: Power Distribution — 7-DoF Arm -> Power Distribution - 7-DoF Arm
