File: hardware/sensor-interface/sensor-interface.kicad_sch (KiCad schematic)
At the start: 7 parts, among them J1 SPI_MCU (shared bus), J2 I2C_MCU, U1 AS5047P (Joint 0), U8 BNO055 (arm base IMU)

Commit message: hardware: regenerate KiCad schematics with correct KiCad 7 syntax
Previous schematics had multiple parser errors:
- (label (text "X") ...) should be (label "X" ...)
- pin instances used names not numbers
- UTF-8 BOM byte from PowerShell Set-Content

Added gen_schematics.py Python generator as source-of-truth.
All three .kicad_sch files now pass: no BOM, starts with '(',
balanced parentheses, correct KiCad 7 S-expression format.

Co-Authored-By: Claude Opus 4.7 (1M context) <noreply@anthropic.com>
Parts:
- removed C1, C3: 100n, symbol C_Decoup
- removed C2: 10u, symbol C_Decoup
- removed J1: SPI_MCU (shared bus), symbol Conn_SPI
- removed J2: I2C_MCU, symbol Conn_I2C
- added J1: SPI_MCU, Connector_PinHeader_2.54mm:PinHeader_1x05_P2.54mm_Vertical, symbol Conn_SPI_5pin
- added J2: I2C_MCU, Connector_PinHeader_2.54mm:PinHeader_1x04_P2.54mm_Vertical, symbol Conn_I2C_4pin
- U1: value AS5047P (Joint 0) -> AS5047P
- U8: value BNO055 (arm base IMU) -> BNO055; footprint Package_LGA:Bosch_LGA-28_5.2x3.8mm_P0.5mm -> Package_LCC:LCC-28_7.0x7.0mm_P0.65mm
Connections:
- net ['text', '+3V3']: no longer names the net of U1.3 (CSn)
- net ['text', 'SPI_CLK']: no longer names the net of U1.1 (VDD3V3)
- net ['text', 'SPI_MISO']: no longer names the net of U1.6 (MISO)
Other:
- note added: "Each encoder uses separate CS line: ENC_CS0..ENC_CS6."
- note added: "NOTE: U2..U7 are identical AS5047P encoders for Joints 1-6."
- title: Sensor Interface — 7-DoF Arm -> Sensor Interface - 7-DoF Arm
Changed lines of the file:
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@@
   (generator "eeschema")
   (generator_version "7.0.11")
-  (paper "A2")
+  (paper "A3")
   (title_block
-    (title "Sensor Interface — 7-DoF Arm")
+    (title "Sensor Interface - 7-DoF Arm")
     (date "2026-05-03")
     (rev "1.0")
     (company "Northeastern University")
-    (comment 1 "AS5047P 14-bit absolute encoder (x7, one per joint) — SPI mode 3")
-    (comment 2 "BNO055 9-DOF IMU — I2C")
-    (comment 3 "Driver: firmware/drivers/as5047p.cpp  |  Interface: hal::IEncoder")
+    (comment 1 "AS5047P 14-bit SPI encoder (x7 joints) + BNO055 I2C IMU")
+    (comment 2 "SPI: 10 MHz / I2C: 400 kHz (Fast-mode)")
   )
-  (symbol (lib_id "Conn_SPI") (at 35 100 0) (unit 1)
+  (symbol (lib_id "Conn_SPI_5pin") (at 50 90 0) (unit 1)
     (in_bom yes) (on_board yes)
-    (property "Reference" "J1" (at 35 90 0) (effects (font (size 1.27 1.27))))
-    (property "Value" "SPI_MCU (shared bus)" (at 35 88 0) (effects (font (size 1.27 1.27))))
-    (pin "MOSI")
-    (pin "MISO")
-    (pin "CLK")
-    (pin "CSn")
-    (pin "3V3")
-  )
-  (symbol (lib_id "AS5047P") (at 100 100 0) (unit 1)
-    (in_bom yes) (on_board yes)
-    (property "Reference" "U1" (at 100 91 0) (effects (font (size 1.27 1.27))))
-    (property "Value" "AS5047P (Joint 0)" (at 100 89 0) (effects (font (size 1.27 1.27))))
-    (property "Footprint" "Package_SO:SOIC-14_3.9x8.7mm_P1.27mm" (at 100 100 0)
+    (property "Reference" "J1" (at 53 88 0)
+      (effects (font (size 1.27 1.27)) (justify left)))
+    (property "Value" "SPI_MCU" (at 53 86 0)
+      (effects (font (size 1.27 1.27)) (justify left)))
+    (property "Footprint" "Connector_PinHeader_2.54mm:PinHeader_1x05_P2.54mm_Vertical" (at 50 90 0)
       (effects (font (size 1.27 1.27)) (hide yes)))
-    (pin "VDD3V3")
-    (pin "GND")
-    (pin "CSn")
-    (pin "CLK")
-    (pin "MOSI")
-    (pin "MISO")
-    (pin "PWM")
-    (pin "DAE")
-  )
-  (symbol (lib_id "C_Decoup") (at 85 97 0) (unit 1)
-    (in_bom yes) (on_board yes)
-    (property "Reference" "C1" (at 88 97 0) (effects (font (size 1.27 1.27))))
-    (property "Value" "100n" (at 88 94.5 0) (effects (font (size 1.27 1.27))))
     (pin "1")
     (pin "2")
+    (pin "3")
+    (pin "4")
+    (pin "5")
   )
-  (symbol (lib_id "C_Decoup") (at 85 107 0) (unit 1)
+  (symbol (lib_id "AS5047P") (at 100 90 0) (unit 1)
     (in_bom yes) (on_board yes)
-    (property "Reference" "C2" (at 88 107 0) (effects (font (size 1.27 1.27))))
-    (property "Value" "10u" (at 88 104.5 0) (effects (font (size 1.27 1.27))))
+    (property "Reference" "U1" (at 103 88 0)
+      (effects (font (size 1.27 1.27)) (justify left)))
+    (property "Value" "AS5047P" (at 103 86 0)
+      (effects (font (size 1.27 1.27)) (justify left)))
+    (property "Footprint" "Package_SO:SOIC-14_3.9x8.7mm_P1.27mm" (at 100 90 0)
+      (effects (font (size 1.27 1.27)) (hide yes)))
     (pin "1")
     (pin "2")
+    (pin "3")
+    (pin "4")
+    (pin "5")
+    (pin "6")
+    (pin "7")
+    (pin "8")
   )
-  (symbol (lib_id "BNO055") (at 100 165 0) (unit 1)
+  (symbol (lib_id "BNO055") (at 100 130 0) (unit 1)
     (in_bom yes) (on_board yes)
-    (property "Reference" "U8" (at 100 154 0) (effects (font (size 1.27 1.27))))
-    (property "Value" "BNO055 (arm base IMU)" (at 100 152 0) (effects (font (size 1.27 1.27))))
-    (property "Footprint" "Package_LGA:Bosch_LGA-28_5.2x3.8mm_P0.5mm" (at 100 165 0)
+    (property "Reference" "U8" (at 103 128 0)
+      (effects (font (size 1.27 1.27)) (justify left)))
+    (property "Value" "BNO055" (at 103 126 0)
+      (effects (font (size 1.27 1.27)) (justify left)))
+    (property "Footprint" "Package_LCC:LCC-28_7.0x7.0mm_P0.65mm" (at 100 130 0)
       (effects (font (size 1.27 1.27)) (hide yes)))
-    (pin "VDD")
-    (pin "VDDIO")
-    (pin "GND")
-    (pin "~{RESET}")
-    (pin "PS0")
-    (pin "PS1")
-    (pin "SDA")
-    (pin "SCL")
-    (pin "INT")
-    (pin "ADR")
-  )
-  (symbol (lib_id "C_Decoup") (at 85 162 0) (unit 1)
-    (in_bom yes) (on_board yes)
-    (property "Reference" "C3" (at 88 162 0) (effects (font (size 1.27 1.27))))
-    (property "Value" "100n" (at 88 159.5 0) (effects (font (size 1.27 1.27))))
     (pin "1")
     (pin "2")
+    (pin "3")
+    (pin "4")
+    (pin "5")
+    (pin "6")
+    (pin "7")
+    (pin "8")
+    (pin "9")
+    (pin "10")
   )
-  (symbol (lib_id "Conn_I2C") (at 35 165 0) (unit 1)
+  (symbol (lib_id "Conn_I2C_4pin") (at 50 130 0) (unit 1)
     (in_bom yes) (on_board yes)
-    (property "Reference" "J2" (at 35 158 0) (effects (font (size 1.27 1.27))))
-    (property "Value" "I2C_MCU" (at 35 156 0) (effects (font (size 1.27 1.27))))
-    (pin "SDA")
-    (pin "SCL")
-    (pin "3V3")
-    (pin "GND")
+    (property "Reference" "J2" (at 53 128 0)
+      (effects (font (size 1.27 1.27)) (justify left)))
+    (property "Value" "I2C_MCU" (at 53 126 0)
+      (effects (font (size 1.27 1.27)) (justify left)))
+    (property "Footprint" "Connector_PinHeader_2.54mm:PinHeader_1x04_P2.54mm_Vertical" (at 50 130 0)
+      (effects (font (size 1.27 1.27)) (hide yes)))
+    (pin "1")
+    (pin "2")
+    (pin "3")
+    (pin "4")
   )
-  (label (text "SPI_MOSI") (at 38.81 106.35 0)
+  (label "SPI_MOSI" (at 75 88 0)
+    (fields_autoplaced yes)
     (effects (font (size 1.27 1.27)) (justify left))
 )
-  (label (text "SPI_MOSI") (at 89.84 102.54 180)
-    (effects (font (size 1.27 1.27)) (justify right))
-)
-  (label (text "SPI_MISO") (at 38.81 103.81 0)
+  (label "SPI_MOSI" (at 85 88 0)
+    (fields_autoplaced yes)
     (effects (font (size 1.27 1.27)) (justify left))
 )
-  (label (text "SPI_MISO") (at 110.16 100 0)
+  (label "SPI_MISO" (at 75 90 0)
+    (fields_autoplaced yes)
     (effects (font (size 1.27 1.27)) (justify left))
 )
-  (label (text "SPI_CLK") (at 38.81 101.27 0)
+  (label "SPI_MISO" (at 85 90 0)
+    (fields_autoplaced yes)
     (effects (font (size 1.27 1.27)) (justify left))
 )
-  (label (text "SPI_CLK") (at 89.84 97.46 180)
-    (effects (font (size 1.27 1.27)) (justify right))
-)
-  (label (text "ENC_CS0") (at 38.81 98.73 0)
+  (label "SPI_CLK" (at 75 92 0)
+    (fields_autoplaced yes)
     (effects (font (size 1.27 1.27)) (justify left))
 )
-  (label (text "ENC_CS0") (at 89.84 94.92 180)
-    (effects (font (size 1.27 1.27)) (justify right))
-)
-  (label (text "+3V3") (at 38.81 96.19 0)
+  (label "SPI_CLK" (at 85 92 0)
+    (fields_autoplaced yes)
     (effects (font (size 1.27 1.27)) (justify left))
 )
-  (label (text "+3V3") (at 89.84 102.54 180)
-    (effects (font (size 1.27 1.27)) (justify right))
-)
-  (label (text "+3V3") (at 38.81 168.81 0)
+  (label "ENC_CS0" (at 75 94 0)
+    (fields_autoplaced yes)
     (effects (font (size 1.27 1.27)) (justify left))
 )
-  (label (text "+3V3") (at 89.84 170.32 180)
-    (effects (font (size 1.27 1.27)) (justify right))
-)
-  (label (text "I2C_SDA") (at 38.81 163.81 0)
+  (label "ENC_CS0" (at 85 94 0)
+    (fields_autoplaced yes)
     (effects (font (size 1.27 1.27)) (justify left))
 )
-  (label (text "I2C_SDA") (at 89.84 170.32 180)
-    (effects (font (size 1.27 1.27)) (justify right))
-)
-  (label (text "I2C_SCL") (at 38.81 161.27 0)
+  (label "+3V3" (at 75 96 0)
+    (fields_autoplaced yes)
     (effects (font (size 1.27 1.27)) (justify left))
 )
-  (label (text "I2C_SCL") (at 110.16 167.78 0)
+  (label "+3V3" (at 85 96 0)
+    (fields_autoplaced yes)
     (effects (font (size 1.27 1.27)) (justify left))
 )
-  (label (text "IMU_INT") (at 110.16 165.24 0)
+  (label "I2C_SDA" (at 75 128 0)
+    (fields_autoplaced yes)
+    (effects (font (size 1.27 1.27)) (justify left))
+)
+  (label "I2C_SDA" (at 85 128 0)
+    (fields_autoplaced yes)
+    (effects (font (size 1.27 1.27)) (justify left))
+)
+  (label "I2C_SCL" (at 75 130 0)
+    (fields_autoplaced yes)
+    (effects (font (size 1.27 1.27)) (justify left))
+)
+  (label "I2C_SCL" (at 85 130 0)
+    (fields_autoplaced yes)
+    (effects (font (size 1.27 1.27)) (justify left))
+)
+  (label "IMU_INT" (at 115 126 0)
+    (fields_autoplaced yes)
+    (effects (font (size 1.27 1.27)) (justify left))
+)
+  (text "NOTE: U2..U7 are identical AS5047P encoders for Joints 1-6." (at 50 75 0)
+    (effects (font (size 1.27 1.27)) (justify left))
+)
+  (text "Each encoder uses separate CS line: ENC_CS0..ENC_CS6." (at 50 72 0)
     (effects (font (size 1.27 1.27)) (justify left))
 )
   (sheet_instances
-    (path "/" (page "1"))
-  )
+    (path "/" (page "1")))
 )
